File: circuit/atmega_multimedia_control.sch (EAGLE design)
At the start: 20 parts, among them IC1 MEGA8-P, Q1 20Mhz, X1 USB

Commit message: fixed schematic
Connections:
- removed net N$5 (its old number): D2.C, R3.1, R4.1, X1.3
- removed net N$6: D1.C, R2.1, X1.2
- new net N$16: D1.C, R2.1, R4.1, X1.2
- new net N$4: D2.C, R3.1, X1.3
Other:
- note added: "D+ (green)"
- note added: "D- (white)"
- moved on the sheet: R2, R3
Changed lines of the file:
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@@
 <text x="147.32" y="38.1" size="1.778" layer="91">button 3</text>
 <text x="88.9" y="78.74" size="1.778" layer="91">volume knob</text>
+<text x="83.82" y="54.61" size="1.524" layer="91" distance="32">D+ (green)</text>
+<text x="83.82" y="41.91" size="1.524" layer="91" distance="32">D- (white)</text>
 </plain>
 <instances>
@@
 <attribute name="VALUE" x="104.902" y="21.971" size="1.778" layer="96"/>
 </instance>
-<instance part="R2" gate="G$1" x="104.14" y="45.72" rot="R180"/>
-<instance part="R3" gate="G$1" x="96.52" y="50.8" rot="R180"/>
+<instance part="R2" gate="G$1" x="96.52" y="45.72" rot="R180"/>
+<instance part="R3" gate="G$1" x="93.98" y="50.8" rot="R180"/>
 <instance part="Q1" gate="G$1" x="25.4" y="58.42" smashed="yes" rot="R90">
 <attribute name="VALUE" x="33.02" y="66.04" size="1.778" layer="96" rot="R180"/>
@@
 </segment>
 </net>
-<net name="N$6" class="0">
-<segment>
-<pinref part="X1" gate="G$1" pin="2"/>
-<wire x1="114.3" y1="5.08" x2="114.3" y2="12.7" width="0.1524" layer="91"/>
-<pinref part="R2" gate="G$1" pin="1"/>
-<wire x1="114.3" y1="12.7" x2="114.3" y2="45.72" width="0.1524" layer="91"/>
-<wire x1="114.3" y1="45.72" x2="109.22" y2="45.72" width="0.1524" layer="91"/>
-<pinref part="D1" gate="G$1" pin="C"/>
-<wire x1="109.22" y1="12.7" x2="114.3" y2="12.7" width="0.1524" layer="91"/>
-<junction x="114.3" y="12.7"/>
-</segment>
-</net>
-<net name="N$4" class="0">
-<segment>
-<pinref part="R2" gate="G$1" pin="2"/>
-<pinref part="IC1" gate="G$1" pin="PD4(XCK/T0)"/>
-<wire x1="99.06" y1="45.72" x2="81.28" y2="45.72" width="0.1524" layer="91"/>
-</segment>
-</net>
-<net name="N$5" class="0">
-<segment>
-<pinref part="R3" gate="G$1" pin="1"/>
-<pinref part="X1" gate="G$1" pin="3"/>
-<wire x1="101.6" y1="50.8" x2="111.76" y2="50.8" width="0.1524" layer="91"/>
-<wire x1="111.76" y1="50.8" x2="111.76" y2="20.32" width="0.1524" layer="91"/>
-<pinref part="R4" gate="G$1" pin="1"/>
-<wire x1="111.76" y1="20.32" x2="111.76" y2="5.08" width="0.1524" layer="91"/>
-<wire x1="104.14" y1="58.42" x2="101.6" y2="58.42" width="0.1524" layer="91"/>
-<wire x1="101.6" y1="58.42" x2="101.6" y2="50.8" width="0.1524" layer="91"/>
-<junction x="101.6" y="50.8"/>
-<pinref part="D2" gate="G$1" pin="C"/>
-<wire x1="109.22" y1="20.32" x2="111.76" y2="20.32" width="0.1524" layer="91"/>
-<junction x="111.76" y="20.32"/>
-</segment>
-</net>
-<net name="N$7" class="0">
-<segment>
-<pinref part="R3" gate="G$1" pin="2"/>
-<pinref part="IC1" gate="G$1" pin="PD2(INT0)"/>
-<wire x1="91.44" y1="50.8" x2="81.28" y2="50.8" width="0.1524" layer="91"/>
-</segment>
-</net>
 <net name="N$8" class="0">
 <segment>
@@
 </segment>
 </net>
+<net name="N$4" class="0">
+<segment>
+<pinref part="X1" gate="G$1" pin="3"/>
+<pinref part="D2" gate="G$1" pin="C"/>
+<wire x1="109.22" y1="20.32" x2="111.76" y2="20.32" width="0.1524" layer="91"/>
+<wire x1="111.76" y1="20.32" x2="111.76" y2="5.08" width="0.1524" layer="91"/>
+<pinref part="R3" gate="G$1" pin="1"/>
+<wire x1="99.06" y1="50.8" x2="111.76" y2="50.8" width="0.1524" layer="91"/>
+<wire x1="111.76" y1="50.8" x2="111.76" y2="20.32" width="0.1524" layer="91"/>
+<junction x="111.76" y="20.32"/>
+</segment>
+</net>
+<net name="N$5" class="0">
+<segment>
+<pinref part="R2" gate="G$1" pin="2"/>
+<pinref part="IC1" gate="G$1" pin="PD4(XCK/T0)"/>
+<wire x1="91.44" y1="45.72" x2="81.28" y2="45.72" width="0.1524" layer="91"/>
+</segment>
+</net>
+<net name="N$7" class="0">
+<segment>
+<pinref part="IC1" gate="G$1" pin="PD2(INT0)"/>
+<pinref part="R3" gate="G$1" pin="2"/>
+<wire x1="81.28" y1="50.8" x2="88.9" y2="50.8" width="0.1524" layer="91"/>
+</segment>
+</net>
+<net name="N$16" class="0">
+<segment>
+<pinref part="D1" gate="G$1" pin="C"/>
+<wire x1="114.3" y1="12.7" x2="109.22" y2="12.7" width="0.1524" layer="91"/>
+<pinref part="X1" gate="G$1" pin="2"/>
+<wire x1="114.3" y1="5.08" x2="114.3" y2="12.7" width="0.1524" layer="91"/>
+<wire x1="114.3" y1="12.7" x2="114.3" y2="45.72" width="0.1524" layer="91"/>
+<pinref part="R4" gate="G$1" pin="1"/>
+<wire x1="104.14" y1="58.42" x2="104.14" y2="45.72" width="0.1524" layer="91"/>
+<pinref part="R2" gate="G$1" pin="1"/>
+<wire x1="104.14" y1="45.72" x2="101.6" y2="45.72" width="0.1524" layer="91"/>
+<wire x1="114.3" y1="45.72" x2="104.14" y2="45.72" width="0.1524" layer="91"/>
+<junction x="104.14" y="45.72"/>
+<junction x="114.3" y="12.7"/>
+</segment>
+</net>
